Commit message: imporve doc and simulation

File: ros2_ws/src/model_description/diff_drive_robot/urdf/diff_drive_robot.xacro (robot description, xacro)
@@ -36,6 +36,6 @@
     </collision>
     <inertial>
-      <mass value="10"/>
-      <xacro:box_inertia m="10" x="0.5" y="0.3" z="0.2"/>
+      <mass value="1"/>
+      <xacro:box_inertia m="1" x="0.5" y="0.3" z="0.2"/>
     </inertial>
   </link>
@@ -51,5 +51,5 @@
         <origin rpy="1.5708 0 0" xyz="0 0 0"/>
         <geometry>
-          <cylinder radius="0.1" length="0.05"></cylinder>
+          <cylinder radius="0.1" length="0.1"></cylinder>
         </geometry>
         <material name="wheel_color">
@@ -60,11 +60,11 @@
         <origin rpy="1.5708 0 0" xyz="0 0 0"/>
         <geometry>
-          <cylinder radius="0.1" length="0.05"></cylinder>
+          <cylinder radius="0.1" length="0.1"></cylinder>
         </geometry>
       </collision>
       <inertial>
         <origin rpy="1.5708 0 0" xyz="0 0 0"/>
-        <mass value="1"/>
-        <xacro:cylinder_inertia m="1" r="0.1" h="0.05"/>
+        <mass value="0.1"/>
+        <xacro:cylinder_inertia m="0.1" r="0.1" h="0.1"/>
       </inertial>
     </link>
@@ -74,36 +74,12 @@
       <child link="${prefix}_wheel"/>
       <origin rpy="0 0 0" xyz="${x} ${y} ${z}"/>
-      <limit effort="100" velocity="100.0"/>
+      <limit effort="1000" velocity="100.0"/>
+      <dynamics damping="0.5"/>
     </joint>
   </xacro:macro>
-  <link name="caster_wheel">
-    <visual>
-      <geometry>
-        <sphere radius="0.05"/>   <!-- 3 cm radius ball -->
-      </geometry>
-      <origin xyz="0 0 0" rpy="0 0 0"/>
-      <material name="gray">
-        <color rgba="0.5 0.5 0.5 1.0"/>
-      </material>
-    </visual>
-    <collision>
-      <geometry>
-        <sphere radius="0.05"/>
-      </geometry>
-      <origin xyz="0 0 0" rpy="0 0 0"/>
-    </collision>
-    <inertial>
-      <mass value="0.1"/>
-      <origin xyz="0 0 0" rpy="0 0 0"/>
-      <inertia ixx="0.0001" iyy="0.0001" izz="0.0001" ixy="0.0" ixz="0.0" iyz="0.0"/>
-    </inertial>
-  </link>
-  <joint name="caster_joint" type="fixed">
-    <parent link="chassis"/>  <!-- your robot's main body -->
-    <child link="caster_wheel"/>
-    <origin xyz="-0.2 0 -0.1" rpy="0 0 0"/>
-  </joint>
   <xacro:wheel prefix="front_left" x="0.2" y="0.2" z="-0.05" />
   <xacro:wheel prefix="front_right" x="0.2" y="-0.2" z="-0.05" />
+  <xacro:wheel prefix="back_left" x="-0.2" y="0.2" z="-0.05" />
+  <xacro:wheel prefix="back_right" x="-0.2" y="-0.2" z="-0.05" />
   <!-- #endregion -->
   <!-- #region: controller -->
